File: pyboard-led-driver.kicad_pcb (KiCad board)
At the start: 2 copper layers, 54 x 64 mm, 23 parts, among them J1 Ch1, J2 Ch2, J3 Ch3, P1 PYBD-WBUS-Host, U1 SN74AHCT125DR

Commit message: Board v1.0
Signed-off-by: Jim Mussared <jim.mussared@gmail.com>
Parts:
- P1: value PYBD-WBUS-Host -> PYBD-WBUS-Adaptor; footprint MicroPython_Pyboard:PYBD_WBUS_Host -> MicroPython_Pyboard:PYBD_WBUS_Adaptor
Routing:
- net DATA3: track 22.7 -> 17.0 mm
- net 5V_1: track 98.5 -> 102.0 mm
- net DATA1: track 24.6 -> 27.4 mm
- net GND: track 12.6 -> 15.3 mm, vias 5 -> 3
- net DATA2: track 22.9 -> 21.6 mm
Other:
- net class Default: clearance 0.2 -> 0.15
- rule trace_clearance: 0.2 -> 0.15
