File: pybd-ws2812-adaptor.kicad_pcb (KiCad board)
At the start: 2 copper layers, 54 x 64 mm, 23 parts, among them J1 Ch1, J2 Ch2, J3 Ch3, P1 PYBD-WBUS-Adaptor, U1 SN74AHCT125DR

Commit message: Rename to pybd-ws2812-adaptor
Signed-off-by: Jim Mussared <jim.mussared@gmail.com>
Other:
- board text added: "github.com/jimmo/pybd-ws2812-adaptor"
- board text removed: "pybd neopixel"

Commit message: Remove ground plane around antenna.
Signed-off-by: Jim Mussared <jim.mussared@gmail.com>
Routing:
- net 5V_1: track 102.0 -> 92.5 mm
- net DATA1: track 27.4 -> 24.9 mm
